File: CD98.kicad_pcb (KiCad board)
At the start: 2 copper layers, 215 parts, among them J1 Conn_01x20, J2 Conn_01x20, SW1 SW_Push, SW2 RotaryEncoder_Switch, U1 ATmega32U4-A, Y1 16MHz

Commit message: v5
Repositioned diodes, wired matrix.
Parts:
- D1, D10, D11, D12, D13, D14, D15, D16, D17, D18, D19, D2, D20, D21, D22, D23, D24, D25, D26, D27, D28, D29, D3, D30, D31, D32, D33, D34, D35, D36, D37, D38, D39, D4, D40, D41, D42, D43, D44, D45, D46, D47, D48, D49, D5, D50, D51, D52, D53, D54, D55, D56, D57, D58, D59, D6, D60, D61, D62, D63, D64, D65, D66, D67, D68, D69, D7, D70, D71, D72, D73, D74, D75, D76, D77, D78, D79, D8, D80, D81, D82, D83, D84, D85, D86, D87, D88, D89, D9, D90, D91, D92, D93, D94, D95, D96, D97, D98: moved to B.Cu
- J1: footprint Connector_PinSocket_2.54mm:PinSocket_1x20_P2.54mm_Horizontal -> Connector_PinSocket_2.00mm:PinSocket_1x20_P2.00mm_Horizontal; moved to F.Cu
- J2: footprint Connector_PinSocket_2.54mm:PinSocket_1x20_P2.54mm_Horizontal -> Connector_PinSocket_2.00mm:PinSocket_1x20_P2.00mm_Horizontal
- moved D85 489.2 mm to (50.8, 48.4), turned to 90 degrees
- moved D86 474.3 mm to (69.8, 48.4), turned to 90 degrees
- moved D87 459.8 mm to (88.9, 48.4), turned to 90 degrees
- moved D88 445.6 mm to (107.9, 48.4), turned to 90 degrees
- moved D75 431.9 mm to (53.2, 200.8), turned to 90 degrees
- moved D89 431.8 mm to (127.0, 48.4), turned to 90 degrees
- moved D17 426.4 mm to (50.8, 124.6), turned to 90 degrees
- moved D1 426.2 mm to (50.8, 105.6), turned to 90 degrees
- moved D32 421.8 mm to (55.6, 143.7), turned to 90 degrees
- moved D47 420.4 mm to (57.9, 162.7), turned to 90 degrees
- moved D90 418.4 mm to (146.0, 48.4), turned to 90 degrees
- moved D61 416.9 mm to (62.7, 181.8), turned to 90 degrees
- moved D2 409.6 mm to (69.8, 105.6), turned to 90 degrees
- moved D18 409.5 mm to (69.8, 124.6), turned to 90 degrees
- moved D76 405.5 mm to (77.0, 200.8), turned to 90 degrees
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Connections:
- J1 pad 1: Net-(J1-Pin_1) -> RE S1
- J1 pad 10: Col 9 -> Col 10
- J1 pad 11: Col 10 -> Col 9
- J1 pad 12: Col 11 -> Col 8
- J1 pad 13: Col 12 -> Col 7
- J1 pad 14: Col 13 -> Net-(J1-Pin_14)
- J1 pad 15: Row 0 -> Col 5
- J1 pad 16: RE A -> Col 4
- J1 pad 17: RE C -> Net-(J1-Pin_17)
- J1 pad 18: RE B -> Col 2
- J1 pad 19: RE S2 -> Net-(J1-Pin_19)
- J1 pad 2: Net-(J1-Pin_2) -> RE S2
- J1 pad 20: RE S1 -> Net-(J1-Pin_20)
- J1 pad 3: Col 2 -> RE B
- J1 pad 4: Net-(J1-Pin_4) -> RE C
- J1 pad 5: Col 4 -> RE A
- J1 pad 6: Col 5 -> Row 0
- J1 pad 7: Net-(J1-Pin_7) -> Col 13
- J1 pad 8: Col 7 -> Col 12
- J1 pad 9: Col 8 -> Col 11
- MX1 pad 1: Net-(J1-Pin_1) -> Net-(J1-Pin_20)
- MX17 pad 1: Net-(J1-Pin_1) -> Net-(J1-Pin_20)
- MX18 pad 1: Net-(J1-Pin_2) -> Net-(J1-Pin_19)
- MX2 pad 1: Net-(J1-Pin_2) -> Net-(J1-Pin_19)
- MX20 pad 1: Net-(J1-Pin_4) -> Net-(J1-Pin_17)
- MX23 pad 1: Net-(J1-Pin_7) -> Net-(J1-Pin_14)
- MX32 pad 1: Net-(J1-Pin_1) -> Net-(J1-Pin_20)
- MX34 pad 1: Net-(J1-Pin_4) -> Net-(J1-Pin_17)
- MX37 pad 1: Net-(J1-Pin_7) -> Net-(J1-Pin_14)
- MX4 pad 1: Net-(J1-Pin_4) -> Net-(J1-Pin_17)
- MX47 pad 1: Net-(J1-Pin_1) -> Net-(J1-Pin_20)
- MX49 pad 1: Net-(J1-Pin_4) -> Net-(J1-Pin_17)
- MX52 pad 1: Net-(J1-Pin_7) -> Net-(J1-Pin_14)
- MX61 pad 1: Net-(J1-Pin_2) -> Net-(J1-Pin_19)
- MX63 pad 1: Net-(J1-Pin_4) -> Net-(J1-Pin_17)
- MX66 pad 1: Net-(J1-Pin_7) -> Net-(J1-Pin_14)
- MX7 pad 1: Net-(J1-Pin_7) -> Net-(J1-Pin_14)
- MX75 pad 1: Net-(J1-Pin_1) -> Net-(J1-Pin_20)
- MX76 pad 1: Net-(J1-Pin_2) -> Net-(J1-Pin_19)
- MX77 pad 1: Net-(J1-Pin_4) -> Net-(J1-Pin_17)
- MX78 pad 1: Net-(J1-Pin_7) -> Net-(J1-Pin_14)
Routing:
- net Net-(J1-Pin_17): track 0.00 -> 110.0 mm
- net Col 10: track 0.00 -> 107.1 mm
- net Col 11: track 0.00 -> 107.1 mm
- net Net-(J1-Pin_14): track 0.00 -> 106.4 mm
- net Net-(J1-Pin_19): track 0.00 -> 106.4 mm
- net Col 13: track 0.00 -> 105.1 mm
- net Col 12: track 0.00 -> 103.7 mm
- net Col 14: track 0.00 -> 103.1 mm
- net Net-(J1-Pin_20): track 0.00 -> 100.2 mm
- net Col 15: track 0.00 -> 95.3 mm
- net Col 8: track 0.00 -> 88.3 mm
- net Col 9: track 0.00 -> 86.1 mm
- net Col 2: track 0.00 -> 86.1 mm
- net Col 5: track 0.00 -> 86.1 mm
- net Col 7: track 0.00 -> 86.1 mm
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